File: pcb/ioExpansion-23017/MCP23017.sch (KiCad schematic (older format))
At the start: 11 parts, among them J1 GS3, J2 GS3, J3 GS3, U1 MCP23017, U2 Header2

Commit message: Improved ioExpansion
Parts:
- added C1: C, Capacitors_THT:C_Disc_D3.8mm_W2.6mm_P2.50mm, symbol C
Connections:
- net labels added: A0, A1, A2, A3, A4, A5, A6, A7, B0, B1, B2, B3, B4, B5, B6, B7, IA, IB
- net labels removed: Earth
Changed lines of the file:
@@
 EESchema Schematic File Version 2
-LIBS:MCP23017-rescue
 LIBS:power
 LIBS:device
@@
 L7
 $Comp
-L Earth #PWR01
-U 1 1 5AC24527
-P 2650 2100
-F 0 "#PWR01" H 2650 1850 50  0001 C CNN
-F 1 "Earth" H 2650 1950 50  0001 C CNN
-F 2 "" H 2650 2100 50  0001 C CNN
-F 3 "" H 2650 2100 50  0001 C CNN
-	1    2650 2100
-	1    0    0    -1
-$EndComp
-$Comp
 L MCP23017 U1
 U 1 1 5AC32B7F
@@
 Wire Wire Line
 	2250 3000 6100 3000
-Connection ~ 2650 2100
 Wire Wire Line
 	4900 5250 5300 5250
@@
 	1    0    0    -1
 $EndComp
-Wire Wire Line
-	3000 4550 3900 4550
-Wire Wire Line
-	3000 4550 3000 3700
-Wire Wire Line
-	3100 3700 3100 4450
-Wire Wire Line
-	3100 4450 3900 4450
-Wire Wire Line
-	3200 3700 3200 4350
-Wire Wire Line
-	3200 4350 3900 4350
-Wire Wire Line
-	3300 3700 3300 4250
-Wire Wire Line
-	3300 4250 3900 4250
-Wire Wire Line
-	3900 4150 3400 4150
-Wire Wire Line
-	3400 4150 3400 3700
-Wire Wire Line
-	3500 3700 3500 4050
-Wire Wire Line
-	3500 4050 3900 4050
-Wire Wire Line
-	3900 3950 3600 3950
-Wire Wire Line
-	3600 3950 3600 3700
-Wire Wire Line
-	3700 3700 3700 3850
-Wire Wire Line
-	3700 3850 3900 3850
-Wire Wire Line
-	3200 5650 3200 5450
-Wire Wire Line
-	3200 5450 3900 5450
-Wire Wire Line
-	3900 5350 3100 5350
-Wire Wire Line
-	3100 5350 3100 5650
-Wire Wire Line
-	3000 5250 3000 5650
-Wire Wire Line
-	3000 5250 3900 5250
-Wire Wire Line
-	3900 5150 2900 5150
-Wire Wire Line
-	2900 5150 2900 5650
-Wire Wire Line
-	2800 5650 2800 5050
-Wire Wire Line
-	2800 5050 3900 5050
-Wire Wire Line
-	3900 4950 2700 4950
-Wire Wire Line
-	2700 4950 2700 5650
-Wire Wire Line
-	2600 5650 2600 4850
-Wire Wire Line
-	2600 4850 3900 4850
-Wire Wire Line
-	3900 4750 2500 4750
-Wire Wire Line
-	2500 4750 2500 5650
+$Comp
+L C C1
+U 1 1 5AE6FD71
+P 4400 3500
+F 0 "C1" H 4425 3600 50  0000 L CNN
+F 1 "C" H 4425 3400 50  0000 L CNN
+F 2 "Capacitors_THT:C_Disc_D3.8mm_W2.6mm_P2.50mm" H 4438 3350 50  0001 C CNN
+F 3 "" H 4400 3500 50  0001 C CNN
+	1    4400 3500
+	1    0    0    -1
+$EndComp
+Text Label 4400 3350 0    60   ~ 0
+GND
+Text Label 4400 3650 0    60   ~ 0
+VCC
+Text Label 4400 5650 0    60   ~ 0
+GND
+Text Label 3450 4750 0    60   ~ 0
+A0
+Text Label 3450 4850 0    60   ~ 0
+A1
+Text Label 3450 4950 0    60   ~ 0
+A2
+Text Label 3450 5050 0    60   ~ 0
+A3
+Text Label 3450 5150 0    60   ~ 0
+A4
+Text Label 3450 5250 0    60   ~ 0
+A5
+Text Label 3450 5350 0    60   ~ 0
+A6
+Text Label 3450 5450 0    60   ~ 0
+A7
+Text Label 3750 3850 0    60   ~ 0
+B0
+Text Label 3750 3950 0    60   ~ 0
+B1
+Text Label 3750 4050 0    60   ~ 0
+B2
+Text Label 3750 4150 0    60   ~ 0
+B3
+Text Label 3750 4250 0    60   ~ 0
+B4
+Text Label 3750 4350 0    60   ~ 0
+B5
+Text Label 3750 4450 0    60   ~ 0
+B6
+Text Label 3750 4550 0    60   ~ 0
+B7
+Wire Wire Line
+	3900 4750 3200 4750
+Wire Wire Line
+	3200 4750 3200 5650
+Wire Wire Line
+	3900 4850 3100 4850
+Wire Wire Line
+	3100 4850 3100 5650
+Wire Wire Line
+	3900 4950 3000 4950
+Wire Wire Line
+	3000 4950 3000 5650
+Wire Wire Line
+	3900 5050 2900 5050
+Wire Wire Line
+	2900 5050 2900 5650
+Wire Wire Line
+	3900 5150 2800 5150
+Wire Wire Line
+	2800 5150 2800 5650
+Wire Wire Line
+	3900 5250 2700 5250
+Wire Wire Line
+	2700 5250 2700 5650
+Wire Wire Line
+	3900 5350 2600 5350
+Wire Wire Line
+	2600 5350 2600 5650
+Wire Wire Line
+	3900 5450 2500 5450
+Wire Wire Line
+	2500 5450 2500 5650
+Wire Wire Line
+	3900 3850 3000 3850
+Wire Wire Line
+	3000 3850 3000 3700
+Wire Wire Line
+	3900 3950 3100 3950
+Wire Wire Line
+	3100 3950 3100 3700
+Wire Wire Line
+	3900 4050 3200 4050
+Wire Wire Line
+	3200 4050 3200 3700
+Wire Wire Line
+	3900 4150 3300 4150
+Wire Wire Line
+	3300 4150 3300 3700
+Wire Wire Line
+	3900 4250 3400 4250
+Wire Wire Line
+	3400 4250 3400 3700
+Wire Wire Line
+	3900 4350 3500 4350
+Wire Wire Line
+	3500 4350 3500 3700
+Wire Wire Line
+	3900 4450 3600 4450
+Wire Wire Line
+	3600 4450 3600 3700
+Wire Wire Line
+	3900 4550 3700 4550
+Wire Wire Line
+	3700 4550 3700 3700
+Text Label 4900 4350 0    60   ~ 0
+IB
+Text Label 4900 4250 0    60   ~ 0
+IA
 $EndSCHEMATC
