File: pcb/levelConverter2/levelConverter.kicad_pcb (KiCad board)
At the start: 2 copper layers, 26 parts, among them Q1 BSS138, Q2 BSS138, Q3 BSS138, Q4 BSS138, Q5 BSS138, Q6 BSS138, Q7 BSS138, Q8 BSS138, U1 AP1117-33

Commit message: Added terminal connectors to the header pins half module. Tweaked the MAX7219 module, and added both common anode and common cathode to stripLED modules.
Parts:
- added J1: S, Pin_Headers:Pin_Header_Straight_1x01_Pitch2.54mm, F.Cu at (164.5, 123.8)
- added J2: Term, Connectors_Terminal_Blocks:TerminalBlock_Pheonix_MPT-2.54mm_3pol, F.Cu at (159.4, 128.9)
- added J3: S, Pin_Headers:Pin_Header_Straight_1x01_Pitch2.54mm, F.Cu at (164.5, 101.0)
- added J4: Term, Connectors_Terminal_Blocks:TerminalBlock_Pheonix_MPT-2.54mm_3pol, F.Cu at (159.4, 90.8)
- H1: value Data -> DATA
Routing:
- net Net-(H3-Pad1): track 40.0 -> 60.3 mm
- net Net-(J3-Pad1): track 0.00 -> 10.2 mm
- net Net-(J1-Pad1): track 0.00 -> 5.08 mm
Other:
- board text added: "G"
- board text added: "V"
