File: pcb/stripLED/stripLED.kicad_pcb (KiCad board)
At the start: 2 copper layers, 34 parts, among them J1 Conn_01x04, J2 Conn_01x03, J6 Conn_01x01, J7 Conn_01x01, J8 Conn_01x04, M3 X, Q1 BSS138, Q2 BSS138, Q3 BSS138, Q4 IRLB8721PBF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

Commit message: Added terminal connectors to the header pins half module. Tweaked the MAX7219 module, and added both common anode and common cathode to stripLED modules.
Parts:
- removed DA1, DA2, DA3, DA4, DA5, DA6, DA7, DA8: DATA, Pin_Headers:Pin_Header_Straight_1x03_Pitch2.54mm
- removed DA10, DA9: DATA, Connectors_Terminal_Blocks:TerminalBlock_Pheonix_MPT-2.54mm_3pol
- removed J6, J7: Conn_01x01, Pin_Headers:Pin_Header_Straight_1x01_Pitch2.54mm
- added H2: Choice, Pin_Headers:Pin_Header_Straight_1x08_Pitch2.54mm, F.Cu at (155.6, 103.5)
- added J3: Select, Pin_Headers:Pin_Header_Straight_1x03_Pitch2.54mm, F.Cu at (158.1, 108.6)
- added J4: Term, Pin_Headers:Pin_Header_Straight_1x04_Pitch2.54mm, F.Cu at (157.5, 86.4)
- added Q10: 2N7002, TO_SOT_Packages_SMD:SOT-23, F.Cu at (157.5, 96.5)
- added Q11: 2N7002, TO_SOT_Packages_SMD:SOT-23, F.Cu at (161.9, 96.5)
- added Q12: 2N7002, TO_SOT_Packages_SMD:SOT-23, F.Cu at (166.4, 96.5)
- added Q7: 2N3904, TO_SOT_Packages_THT:TO-92_Molded_Narrow, F.Cu at (163.8, 116.2)
- added Q8: 2N3904, TO_SOT_Packages_THT:TO-92_Molded_Narrow, F.Cu at (163.8, 109.9)
- added Q9: 2N3904, TO_SOT_Packages_THT:TO-92_Molded_Narrow, F.Cu at (163.8, 103.5)
- added R1: 10K, Resistors_THT:R_Axial_DIN0204_L3.6mm_D1.6mm_P7.62mm_Horizontal, F.Cu at (160.0, 121.3)
- added R2: 10K, Resistors_THT:R_Axial_DIN0204_L3.6mm_D1.6mm_P7.62mm_Horizontal, F.Cu at (163.2, 121.3)
- added R3: 10K, Resistors_THT:R_Axial_DIN0204_L3.6mm_D1.6mm_P7.62mm_Horizontal, F.Cu at (165.7, 121.3)
- added RN1: 10K, Resistors_THT:R_Array_SIP5, F.Cu at (156.8, 90.8)
- H1: value Headers8L -> Choice
- J1, J8: value Conn_01x04 -> Term
- J2: value Conn_01x03 -> Select
Routing:
- net /VCC2: track 59.7 -> 17.1 mm, vias 1 -> 0
- net Net-(Q10-Pad1): track 0.00 -> 31.8 mm, vias 0 -> 1
- net Net-(J3-Pad1): track 0.00 -> 25.1 mm
- net Net-(Q11-Pad1): track 0.00 -> 22.8 mm, vias 0 -> 1
- net Net-(Q9-Pad2): track 0.00 -> 22.5 mm
- net Net-(J3-Pad2): track 0.00 -> 20.9 mm
- net Net-(J3-Pad3): track 0.00 -> 16.8 mm
- net Net-(Q8-Pad2): track 0.00 -> 16.2 mm
- net Net-(DA10-Pad3): track 14.6 -> 0.00 mm
- net Net-(Q12-Pad1): track 0.00 -> 13.9 mm
- net Net-(J4-Pad2): track 0.00 -> 12.3 mm
- net Net-(J4-Pad4): track 0.00 -> 12.1 mm
- net Net-(J4-Pad3): track 0.00 -> 11.6 mm
- net /VIN2: track 17.1 -> 28.5 mm, vias 0 -> 3
- net Net-(Q7-Pad2): track 0.00 -> 9.57 mm
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Other:
- board text added: "+"
- board text added: "RGB LED v1.0"
- board text added: "nickthecoder.co.uk"
- board text removed: "DATA"
- board text removed: "Header Module v1.0"
- board text removed: "RGB LED Module v1.0"
- board text removed: "VCC"
- board text removed: "http://nickthecoder.co.uk"

Commit message: Tweaked the stripLED module.
Parts:
- removed R1, R2, R3: 10K, Resistors_THT:R_Axial_DIN0204_L3.6mm_D1.6mm_P7.62mm_Horizontal
- Q7, Q8, Q9: value 2N3904 -> BSS83P; footprint TO_SOT_Packages_THT:TO-92_Molded_Narrow -> TO_SOT_Packages_SMD:SOT-23
- moved Q7 17.7 mm to (157.5, 99.7), turned to 90 degrees
- moved Q8 10.3 mm to (161.9, 99.7), turned to 90 degrees
- moved Q10 5.85 mm to (156.2, 90.8)
- moved Q11 5.75 mm to (161.3, 90.8)
- moved Q12 5.71 mm to (166.4, 90.8)
- moved RN1 5.12 mm to (156.2, 95.9)
- moved Q9 4.58 mm to (166.4, 99.7), turned to 90 degrees
Connections:
- net Net-(Q10-Pad1) renamed /gate4
- net Net-(Q11-Pad1) renamed /gate5
- net Net-(Q12-Pad1) renamed /gate6
- J3 pad 1: Net-(J3-Pad1) -> /gate1
- J3 pad 2: Net-(J3-Pad2) -> /gate2
- J3 pad 3: Net-(J3-Pad3) -> /gate3
- Q7 pad 1: /GND2 -> /gate1
- Q7 pad 2: Net-(Q7-Pad2) -> /GND2
- Q8 pad 1: /GND2 -> /gate2
- Q8 pad 2: Net-(Q8-Pad2) -> /GND2
- Q9 pad 1: /GND2 -> /gate3
- Q9 pad 2: Net-(Q9-Pad2) -> /GND2
Routing:
- net Net-(J3-Pad1): track 25.1 -> 0.00 mm
- net /gate4: track 31.8 -> 8.86 mm, vias 1 -> 0
- net Net-(Q9-Pad2): track 22.5 -> 0.00 mm
- net Net-(J3-Pad2): track 20.9 -> 0.00 mm
- net Net-(J3-Pad3): track 16.8 -> 0.00 mm
- net Net-(Q8-Pad2): track 16.2 -> 0.00 mm
- net /gate3: track 0.00 -> 16.0 mm
- net /gate5: track 22.8 -> 7.55 mm, vias 1 -> 0
- net /gate2: track 0.00 -> 11.6 mm
- net Net-(Q7-Pad2): track 9.57 -> 0.00 mm
- net /gate1: track 0.00 -> 8.55 mm
- net /GND2: track 0.00 -> 7.54 mm, vias 0 -> 3
- net Net-(J4-Pad3): track 11.6 -> 5.58 mm
- net Net-(J4-Pad4): track 12.1 -> 6.36 mm
- net Net-(J4-Pad2): track 12.3 -> 6.63 mm
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Other:
- board text added: "A"
- board text added: "B"
- board text added: "C"
- board text added: "G"
- board text added: "RGB LED"
