File: pcb/wemos/wemos.kicad_pcb (KiCad board)
At the start: 2 copper layers, 9 parts, among them SW1 SW_SPST, U1 wemos

Commit message: Added a Rotary Encoder module. Tidied up a couple of modules before printing them.
Other:
- board text added: "WeMos v1.0 nickthecoder.co.uk"
- board text removed: "WeMos v1.0 http://nickthecoder.co.uk"
Changed lines of the file:
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@@
   )
   (setup
-    (last_trace_width 0.5)
+    (last_trace_width 0.25)
     (user_trace_width 0.5)
     (trace_clearance 0.2)
@@
     (descr "Through hole straight socket strip, 1x12, 2.54mm pitch, single row")
     (tags "Through hole socket strip THT 1x12 2.54mm single row")
-    (fp_text reference O1 (at 0 -2.33) (layer F.SilkS)
+    (fp_text reference O1 (at 0 -2.33) (layer F.Fab)
       (effects (font (size 1 1) (thickness 0.15)))
     )
@@
     (fp_line (start 1.8 29.75) (end 1.8 -1.8) (layer F.CrtYd) (width 0.05))
     (fp_line (start 1.8 -1.8) (end -1.8 -1.8) (layer F.CrtYd) (width 0.05))
-    (fp_text user %R (at 0 -2.33) (layer F.Fab)
+    (fp_text user %R (at 0 -2.33) (layer F.Fab) hide
       (effects (font (size 1 1) (thickness 0.15)))
     )
@@
     (descr "Through hole straight socket strip, 1x12, 2.54mm pitch, single row")
     (tags "Through hole socket strip THT 1x12 2.54mm single row")
-    (fp_text reference I1 (at 0 -2.33) (layer F.SilkS)
+    (fp_text reference I1 (at 0 -2.33) (layer F.Fab)
       (effects (font (size 1 1) (thickness 0.15)))
     )
@@
     (fp_line (start 1.8 29.75) (end 1.8 -1.8) (layer F.CrtYd) (width 0.05))
     (fp_line (start 1.8 -1.8) (end -1.8 -1.8) (layer F.CrtYd) (width 0.05))
-    (fp_text user %R (at 0 -2.33) (layer F.Fab)
+    (fp_text user %R (at 0 -2.33) (layer F.Fab) hide
       (effects (font (size 1 1) (thickness 0.15)))
     )
@@
     (effects (font (size 1 1) (thickness 0.2)) (justify left))
   )
-  (gr_text "WeMos v1.0\nhttp://nickthecoder.co.uk" (at 135.255 128.27) (layer F.SilkS)
+  (gr_text "WeMos v1.0\nnickthecoder.co.uk" (at 135.255 128.27) (layer F.SilkS)
     (effects (font (size 1.5 1.5) (thickness 0.3)) (justify left))
   )
