File: bluePill/bluePill.sch (KiCad schematic (older format))
At the start: 9 parts, among them J1 Header2, J2 Header1, J3 Power, U1 BluePill

Commit message: Began fixing eplay component library, and schematics, so that the power pins don't issue warnings.
Connections:
- net B14: now also J1.3 (Pin_3)
Changed lines of the file:
@@
 LIBS:valves
 LIBS:eplay
-LIBS:arduino
 LIBS:bluePill-cache
 EELAYER 25 0
@@
 Text Label 1950 1150 2    60   ~ 0
 B12
-Wire Wire Line
-	1050 2550 1950 2550
-Wire Wire Line
-	1050 2450 1950 2450
 Text Label 1350 1650 2    60   ~ 0
 TX1
 Text Label 1350 1750 2    60   ~ 0
 RX1
-Wire Wire Line
-	1050 1650 1950 1650
-Wire Wire Line
-	1050 1750 1950 1750
 Text Label 3250 2350 0    60   ~ 0
 RX2
 Text Label 3250 2450 0    60   ~ 0
 TX2
-Wire Wire Line
-	2850 2350 3850 2350
-Wire Wire Line
-	2850 2450 3850 2450
 Text Label 9000 2050 2    60   ~ 0
 A6
@@
 Text Label 1350 1250 2    60   ~ 0
 SCK2
-Wire Wire Line
-	1050 1250 1950 1250
-Wire Wire Line
-	1950 1350 1350 1350
-Wire Wire Line
-	1050 1450 1950 1450
 $Comp
 L Output O4
@@
 Text Label 8100 4400 2    60   ~ 0
 RX2
-Wire Wire Line
-	2850 2150 3850 2150
-Wire Wire Line
-	2850 1950 3850 1950
-Wire Wire Line
-	2850 2050 3850 2050
 Text Label 7900 2150 2    60   ~ 0
 A11
@@
 Text Label 3250 1550 0    60   ~ 0
 SDA2
-Wire Wire Line
-	2850 1550 3850 1550
-Wire Wire Line
-	2850 1650 3850 1650
 Text Label 1400 2450 2    60   ~ 0
 SCL1
@@
 	1    0    0    -1
 $EndComp
-Wire Wire Line
-	2850 1150 3850 1150
-Wire Wire Line
-	3850 1250 2850 1250
-Wire Wire Line
-	2850 1350 3850 1350
-Wire Wire Line
-	3850 1450 2850 1450
-Wire Wire Line
-	3850 1750 2850 1750
-Wire Wire Line
-	2850 1850 3850 1850
-Wire Wire Line
-	2850 2250 3850 2250
-Wire Wire Line
-	3850 2550 2850 2550
-Wire Wire Line
-	2850 2650 3850 2650
-Wire Wire Line
-	3850 2750 2850 2750
-Wire Wire Line
-	2850 2850 3850 2850
-Wire Wire Line
-	3850 2950 2850 2950
-Wire Wire Line
-	2850 3050 3850 3050
 $Comp
 L Conn_01x20 J1
@@
 	-1   0    0    -1
 $EndComp
-Wire Wire Line
-	1950 1150 1050 1150
-Wire Wire Line
-	1300 1350 1050 1350
-Wire Wire Line
-	1050 1550 1950 1550
-Wire Wire Line
-	1050 1850 1950 1850
-Wire Wire Line
-	1950 1950 1050 1950
-Wire Wire Line
-	1050 2050 1950 2050
-Wire Wire Line
-	1950 2150 1050 2150
-Wire Wire Line
-	1050 2250 1950 2250
-Wire Wire Line
-	1950 2350 1050 2350
-Wire Wire Line
-	1050 2650 1950 2650
-Wire Wire Line
-	1950 2750 1050 2750
-Wire Wire Line
-	1050 2850 1950 2850
-Wire Wire Line
-	1950 2950 1050 2950
-Wire Wire Line
-	1050 3050 1950 3050
 Text Label 7900 1650 2    60   ~ 0
 VCC
@@
 	1    0    0    -1
 $EndComp
+Wire Wire Line
+	1050 2550 1950 2550
+Wire Wire Line
+	1050 2450 1950 2450
+Wire Wire Line
+	1050 1650 1950 1650
+Wire Wire Line
+	1050 1750 1950 1750
+Wire Wire Line
+	2850 2350 3850 2350
+Wire Wire Line
+	2850 2450 3850 2450
+Wire Wire Line
+	1050 1250 1950 1250
+Wire Wire Line
+	1050 1350 1950 1350
+Wire Wire Line
+	1050 1450 1950 1450
+Wire Wire Line
+	2850 2150 3850 2150
+Wire Wire Line
+	2850 1950 3850 1950
+Wire Wire Line
+	2850 2050 3850 2050
+Wire Wire Line
+	2850 1550 3850 1550
+Wire Wire Line
+	2850 1650 3850 1650
+Wire Wire Line
+	2850 1150 3850 1150
+Wire Wire Line
+	3850 1250 2850 1250
+Wire Wire Line
+	2850 1350 3850 1350
+Wire Wire Line
+	3850 1450 2850 1450
+Wire Wire Line
+	3850 1750 2850 1750
+Wire Wire Line
+	2850 1850 3850 1850
+Wire Wire Line
+	2850 2250 3850 2250
+Wire Wire Line
+	3850 2550 2850 2550
+Wire Wire Line
+	2850 2650 3850 2650
+Wire Wire Line
+	3850 2750 2850 2750
+Wire Wire Line
+	2850 2850 3850 2850
+Wire Wire Line
+	3850 2950 2850 2950
+Wire Wire Line
+	2850 3050 3850 3050
+Wire Wire Line
+	1950 1150 1050 1150
+Wire Wire Line
+	1050 1550 1950 1550
+Wire Wire Line
+	1050 1850 1950 1850
+Wire Wire Line
+	1950 1950 1050 1950
+Wire Wire Line
+	1050 2050 1950 2050
+Wire Wire Line
+	1950 2150 1050 2150
+Wire Wire Line
+	1050 2250 1950 2250
+Wire Wire Line
+	1950 2350 1050 2350
+Wire Wire Line
+	1050 2650 1950 2650
+Wire Wire Line
+	1950 2750 1050 2750
+Wire Wire Line
+	1050 2850 1950 2850
+Wire Wire Line
+	1950 2950 1050 2950
+Wire Wire Line
+	1050 3050 1950 3050
+$Comp
+L PWR_FLAG #FLG01
+U 1 1 5AFEA06F
+P 4650 3300
+F 0 "#FLG01" H 4650 3375 50  0001 C CNN
+F 1 "PWR_FLAG" H 4650 3450 50  0000 C CNN
+F 2 "" H 4650 3300 50  0001 C CNN
+F 3 "" H 4650 3300 50  0001 C CNN
+	1    4650 3300
+	1    0    0    -1
+$EndComp
+Wire Wire Line
+	5100 3350 4650 3350
+Wire Wire Line
+	4650 3350 4650 3300
+$Comp
+L PWR_FLAG #FLG02
+U 1 1 5AFEA32E
+P 6650 1550
+F 0 "#FLG02" H 6650 1625 50  0001 C CNN
+F 1 "PWR_FLAG" H 6650 1700 50  0000 C CNN
+F 2 "" H 6650 1550 50  0001 C CNN
+F 3 "" H 6650 1550 50  0001 C CNN
+	1    6650 1550
+	1    0    0    -1
+$EndComp
+Wire Wire Line
+	7050 1550 6650 1550
 $EndSCHEMATC
