File: TM1637/TM1637.kicad_pcb (KiCad board)
At the start: 2 copper layers, 22 parts, among them J1 Conn_01x02, J2 Conn_01x08, J3 Conn_01x06, SW1 SW_SPST, SW2 SW_SPST, SW3 SW_SPST, SW4 SW_SPST, SW5 SW_SPST, SW6 SW_SPST, SW7 SW_SPST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

Commit message: More work to ensure there are no errors from KiCAD's schematic checker. Fixed the multiplexer module, so that all 7 slaves will work (only 6 were working, due to a missing VCC to the "Next Output").
Parts:
- removed H1: Headers8L, Pin_Headers:Pin_Header_Straight_1x08_Pitch2.54mm
- added J4: Choice, Pin_Headers:Pin_Header_Straight_1x08_Pitch2.54mm, F.Cu at (131.4, 103.5)
- J1: value Conn_01x02 -> Select
- J2: value Conn_01x08 -> Segments
- J3: value Conn_01x06 -> Grids
Connections:
- net Earth renamed /GND
Other:
- board text added: "TM1637 v1.1 http://nickthecoder.co.uk"
- board text removed: "MAX7219 v1.1 http://nickthecoder.co.uk"
