File: blank/blank.kicad_pcb (KiCad board)
At the start: 2 copper layers, 6 parts

Commit message: More work to ensure there are no errors from KiCAD's schematic checker. Fixed the multiplexer module, so that all 7 slaves will work (only 6 were working, due to a missing VCC to the "Next Output").
Connections:
- net Earth renamed /GND
Changed lines of the file:
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@@
     (links 11)
     (no_connects 0)
-    (area 124.46 82.55 173.990001 132.080001)
+    (area 0 0 0 0)
     (thickness 1.6)
     (drawings 1)
@@
   (net 1 /VIN)
   (net 2 /VCC)
-  (net 3 Earth)
-  (net 4 /L0)
-  (net 5 /L1)
-  (net 6 /L2)
-  (net 7 /L3)
-  (net 8 /L4)
-  (net 9 /L5)
-  (net 10 /L6)
-  (net 11 /L7)
+  (net 3 /L0)
+  (net 4 /L1)
+  (net 5 /L2)
+  (net 6 /L3)
+  (net 7 /L4)
+  (net 8 /L5)
+  (net 9 /L6)
+  (net 10 /L7)
+  (net 11 /GND)
   (net_class Default "This is the default net class."
     (clearance 0.2)
@@
     (uvia_dia 0.3)
     (uvia_drill 0.1)
+    (add_net /GND)
     (add_net /L0)
     (add_net /L1)
@@
     (add_net /VCC)
     (add_net /VIN)
-    (add_net Earth)
   )
   (module Mounting_Holes:MountingHole_3.2mm_M3 (layer F.Cu)
@@
       (net 2 /VCC))
     (pad 3 thru_hole oval (at 0 5.08) (size 1.7 1.7) (drill 1) (layers *.Cu *.Mask)
-      (net 3 Earth))
+      (net 11 /GND))
     (pad 4 thru_hole oval (at 0 7.62) (size 1.7 1.7) (drill 1) (layers *.Cu *.Mask))
     (pad 5 thru_hole oval (at 0 10.16) (size 1.7 1.7) (drill 1) (layers *.Cu *.Mask)
-      (net 4 /L0))
+      (net 3 /L0))
     (pad 6 thru_hole oval (at 0 12.7) (size 1.7 1.7) (drill 1) (layers *.Cu *.Mask)
-      (net 5 /L1))
+      (net 4 /L1))
     (pad 7 thru_hole oval (at 0 15.24) (size 1.7 1.7) (drill 1) (layers *.Cu *.Mask)
-      (net 6 /L2))
+      (net 5 /L2))
     (pad 8 thru_hole oval (at 0 17.78) (size 1.7 1.7) (drill 1) (layers *.Cu *.Mask)
-      (net 7 /L3))
+      (net 6 /L3))
     (pad 9 thru_hole oval (at 0 20.32) (size 1.7 1.7) (drill 1) (layers *.Cu *.Mask)
-      (net 8 /L4))
+      (net 7 /L4))
     (pad 10 thru_hole oval (at 0 22.86) (size 1.7 1.7) (drill 1) (layers *.Cu *.Mask)
-      (net 9 /L5))
+      (net 8 /L5))
     (pad 11 thru_hole oval (at 0 25.4) (size 1.7 1.7) (drill 1) (layers *.Cu *.Mask)
-      (net 10 /L6))
+      (net 9 /L6))
     (pad 12 thru_hole oval (at 0 27.94) (size 1.7 1.7) (drill 1) (layers *.Cu *.Mask)
-      (net 11 /L7))
+      (net 10 /L7))
     (model ${KISYS3DMOD}/Pin_Headers.3dshapes/Pin_Header_Straight_1x12_Pitch2.54mm.wrl
       (at (xyz 0 0 0))
@@
       (net 2 /VCC))
     (pad 3 thru_hole oval (at 0 5.08) (size 1.7 1.7) (drill 1) (layers *.Cu *.Mask)
-      (net 3 Earth))
+      (net 11 /GND))
     (pad 4 thru_hole oval (at 0 7.62) (size 1.7 1.7) (drill 1) (layers *.Cu *.Mask))
     (pad 5 thru_hole oval (at 0 10.16) (size 1.7 1.7) (drill 1) (layers *.Cu *.Mask)
-      (net 4 /L0))
+      (net 3 /L0))
     (pad 6 thru_hole oval (at 0 12.7) (size 1.7 1.7) (drill 1) (layers *.Cu *.Mask)
-      (net 5 /L1))
+      (net 4 /L1))
     (pad 7 thru_hole oval (at 0 15.24) (size 1.7 1.7) (drill 1) (layers *.Cu *.Mask)
-      (net 6 /L2))
+      (net 5 /L2))
     (pad 8 thru_hole oval (at 0 17.78) (size 1.7 1.7) (drill 1) (layers *.Cu *.Mask)
-      (net 7 /L3))
+      (net 6 /L3))
     (pad 9 thru_hole oval (at 0 20.32) (size 1.7 1.7) (drill 1) (layers *.Cu *.Mask)
-      (net 8 /L4))
+      (net 7 /L4))
     (pad 10 thru_hole oval (at 0 22.86) (size 1.7 1.7) (drill 1) (layers *.Cu *.Mask)
-      (net 9 /L5))
+      (net 8 /L5))
     (pad 11 thru_hole oval (at 0 25.4) (size 1.7 1.7) (drill 1) (layers *.Cu *.Mask)
-      (net 10 /L6))
+      (net 9 /L6))
     (pad 12 thru_hole oval (at 0 27.94) (size 1.7 1.7) (drill 1) (layers *.Cu *.Mask)
-      (net 11 /L7))
+      (net 10 /L7))
     (model ${KISYS3DMOD}/Socket_Strips.3dshapes/Socket_Strip_Straight_1x12_Pitch2.54mm.wrl
       (at (xyz 0 -0.55 0))
@@
   (segment (start 158.115 85.725) (end 168.275 95.885) (width 0.5) (layer F.Cu) (net 2))
   (segment (start 129.54 95.885) (end 139.7 85.725) (width 0.5) (layer F.Cu) (net 2))
-  (segment (start 128.27 103.505) (end 170.18 103.505) (width 0.25) (layer F.Cu) (net 4))
-  (segment (start 128.27 106.045) (end 170.18 106.045) (width 0.25) (layer F.Cu) (net 5))
-  (segment (start 170.18 108.585) (end 128.27 108.585) (width 0.25) (layer F.Cu) (net 6))
-  (segment (start 128.27 111.125) (end 170.18 111.125) (width 0.25) (layer F.Cu) (net 7))
-  (segment (start 170.18 113.665) (end 128.27 113.665) (width 0.25) (layer F.Cu) (net 8))
-  (segment (start 128.27 116.205) (end 170.18 116.205) (width 0.25) (layer F.Cu) (net 9))
-  (segment (start 170.18 118.745) (end 128.27 118.745) (width 0.25) (layer F.Cu) (net 10))
-  (segment (start 128.27 121.285) (end 170.18 121.285) (width 0.25) (layer F.Cu) (net 11))
+  (segment (start 128.27 103.505) (end 170.18 103.505) (width 0.25) (layer F.Cu) (net 3))
+  (segment (start 128.27 106.045) (end 170.18 106.045) (width 0.25) (layer F.Cu) (net 4))
+  (segment (start 170.18 108.585) (end 128.27 108.585) (width 0.25) (layer F.Cu) (net 5))
+  (segment (start 128.27 111.125) (end 170.18 111.125) (width 0.25) (layer F.Cu) (net 6))
+  (segment (start 170.18 113.665) (end 128.27 113.665) (width 0.25) (layer F.Cu) (net 7))
+  (segment (start 128.27 116.205) (end 170.18 116.205) (width 0.25) (layer F.Cu) (net 8))
+  (segment (start 170.18 118.745) (end 128.27 118.745) (width 0.25) (layer F.Cu) (net 9))
+  (segment (start 128.27 121.285) (end 170.18 121.285) (width 0.25) (layer F.Cu) (net 10))
   (zone (net 0) (net_name "") (layer Edge.Cuts) (hatch edge 0.508)
     (connect_pads (clearance 0.508))
@@
     )
   )
-  (zone (net 3) (net_name Earth) (layer B.Cu) (hatch edge 0.508)
+  (zone (net 11) (net_name /GND) (layer B.Cu) (hatch edge 0.508)
     (connect_pads (clearance 0.508))
     (min_thickness 0.254)
