File: blankHalf/blankHalf.kicad_pcb (KiCad board)
At the start: 2 copper layers, 12 parts

Commit message: More work to ensure there are no errors from KiCAD's schematic checker. Fixed the multiplexer module, so that all 7 slaves will work (only 6 were working, due to a missing VCC to the "Next Output").
Connections:
- net Earth renamed /GND
Changed lines of the file:
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@@
   (general
     (links 22)
-    (no_connects 22)
+    (no_connects 20)
     (area 0 0 0 0)
     (thickness 1.6)
@@
   (net 1 /VIN)
   (net 2 /VCC)
-  (net 3 Earth)
-  (net 4 /L0)
-  (net 5 /L1)
-  (net 6 /L2)
-  (net 7 /L3)
-  (net 8 /L4)
-  (net 9 /L5)
-  (net 10 /L6)
-  (net 11 /L7)
-  (net 12 /D0)
-  (net 13 /D1)
-  (net 14 /D2)
-  (net 15 /D3)
-  (net 16 /D4)
-  (net 17 /D5)
-  (net 18 /D6)
-  (net 19 /D7)
-  (net 20 /VIN2)
-  (net 21 /VCC2)
-  (net 22 /GND2)
+  (net 3 /L0)
+  (net 4 /L1)
+  (net 5 /L2)
+  (net 6 /L3)
+  (net 7 /L4)
+  (net 8 /L5)
+  (net 9 /L6)
+  (net 10 /L7)
+  (net 11 /D0)
+  (net 12 /D1)
+  (net 13 /D2)
+  (net 14 /D3)
+  (net 15 /D4)
+  (net 16 /D5)
+  (net 17 /D6)
+  (net 18 /D7)
+  (net 19 /VIN2)
+  (net 20 /VCC2)
+  (net 21 /GND2)
+  (net 22 /GND)
   (net_class Default "This is the default net class."
     (clearance 0.2)
@@
     (add_net /D6)
     (add_net /D7)
+    (add_net /GND)
     (add_net /GND2)
     (add_net /L0)
@@
     (add_net /VIN)
     (add_net /VIN2)
-    (add_net Earth)
   )
   (module Mounting_Holes:MountingHole_3.2mm_M3 (layer F.Cu)
@@
       (net 2 /VCC))
     (pad 3 thru_hole oval (at 0 5.08) (size 1.7 1.7) (drill 1) (layers *.Cu *.Mask)
-      (net 3 Earth))
+      (net 22 /GND))
     (pad 4 thru_hole oval (at 0 7.62) (size 1.7 1.7) (drill 1) (layers *.Cu *.Mask))
     (pad 5 thru_hole oval (at 0 10.16) (size 1.7 1.7) (drill 1) (layers *.Cu *.Mask)
-      (net 4 /L0))
+      (net 3 /L0))
     (pad 6 thru_hole oval (at 0 12.7) (size 1.7 1.7) (drill 1) (layers *.Cu *.Mask)
-      (net 5 /L1))
+      (net 4 /L1))
     (pad 7 thru_hole oval (at 0 15.24) (size 1.7 1.7) (drill 1) (layers *.Cu *.Mask)
-      (net 6 /L2))
+      (net 5 /L2))
     (pad 8 thru_hole oval (at 0 17.78) (size 1.7 1.7) (drill 1) (layers *.Cu *.Mask)
-      (net 7 /L3))
+      (net 6 /L3))
     (pad 9 thru_hole oval (at 0 20.32) (size 1.7 1.7) (drill 1) (layers *.Cu *.Mask)
-      (net 8 /L4))
+      (net 7 /L4))
     (pad 10 thru_hole oval (at 0 22.86) (size 1.7 1.7) (drill 1) (layers *.Cu *.Mask)
-      (net 9 /L5))
+      (net 8 /L5))
     (pad 11 thru_hole oval (at 0 25.4) (size 1.7 1.7) (drill 1) (layers *.Cu *.Mask)
-      (net 10 /L6))
+      (net 9 /L6))
     (pad 12 thru_hole oval (at 0 27.94) (size 1.7 1.7) (drill 1) (layers *.Cu *.Mask)
-      (net 11 /L7))
+      (net 10 /L7))
     (model ${KISYS3DMOD}/Pin_Headers.3dshapes/Pin_Header_Straight_1x12_Pitch2.54mm.wrl
       (at (xyz 0 0 0))
@@
     )
     (pad 1 thru_hole rect (at 0 0) (size 1.7 1.7) (drill 1) (layers *.Cu *.Mask)
-      (net 20 /VIN2))
+      (net 19 /VIN2))
     (pad 2 thru_hole oval (at 0 2.54) (size 1.7 1.7) (drill 1) (layers *.Cu *.Mask)
-      (net 21 /VCC2))
+      (net 20 /VCC2))
     (pad 3 thru_hole oval (at 0 5.08) (size 1.7 1.7) (drill 1) (layers *.Cu *.Mask)
-      (net 22 /GND2))
+      (net 21 /GND2))
     (pad 4 thru_hole oval (at 0 7.62) (size 1.7 1.7) (drill 1) (layers *.Cu *.Mask))
     (pad 5 thru_hole oval (at 0 10.16) (size 1.7 1.7) (drill 1) (layers *.Cu *.Mask)
-      (net 12 /D0))
+      (net 11 /D0))
     (pad 6 thru_hole oval (at 0 12.7) (size 1.7 1.7) (drill 1) (layers *.Cu *.Mask)
-      (net 13 /D1))
+      (net 12 /D1))
     (pad 7 thru_hole oval (at 0 15.24) (size 1.7 1.7) (drill 1) (layers *.Cu *.Mask)
-      (net 14 /D2))
+      (net 13 /D2))
     (pad 8 thru_hole oval (at 0 17.78) (size 1.7 1.7) (drill 1) (layers *.Cu *.Mask)
-      (net 15 /D3))
+      (net 14 /D3))
     (pad 9 thru_hole oval (at 0 20.32) (size 1.7 1.7) (drill 1) (layers *.Cu *.Mask)
-      (net 16 /D4))
+      (net 15 /D4))
     (pad 10 thru_hole oval (at 0 22.86) (size 1.7 1.7) (drill 1) (layers *.Cu *.Mask)
-      (net 17 /D5))
+      (net 16 /D5))
     (pad 11 thru_hole oval (at 0 25.4) (size 1.7 1.7) (drill 1) (layers *.Cu *.Mask)
-      (net 18 /D6))
+      (net 17 /D6))
     (pad 12 thru_hole oval (at 0 27.94) (size 1.7 1.7) (drill 1) (layers *.Cu *.Mask)
-      (net 19 /D7))
+      (net 18 /D7))
     (model ${KISYS3DMOD}/Pin_Headers.3dshapes/Pin_Header_Straight_1x12_Pitch2.54mm.wrl
       (at (xyz 0 0 0))
@@
       (net 2 /VCC))
     (pad 3 thru_hole oval (at 0 5.08) (size 1.7 1.7) (drill 1) (layers *.Cu *.Mask)
-      (net 3 Earth))
+      (net 22 /GND))
     (pad 4 thru_hole oval (at 0 7.62) (size 1.7 1.7) (drill 1) (layers *.Cu *.Mask))
     (pad 5 thru_hole oval (at 0 10.16) (size 1.7 1.7) (drill 1) (layers *.Cu *.Mask)
-      (net 4 /L0))
+      (net 3 /L0))
     (pad 6 thru_hole oval (at 0 12.7) (size 1.7 1.7) (drill 1) (layers *.Cu *.Mask)
-      (net 5 /L1))
+      (net 4 /L1))
     (pad 7 thru_hole oval (at 0 15.24) (size 1.7 1.7) (drill 1) (layers *.Cu *.Mask)
-      (net 6 /L2))
+      (net 5 /L2))
     (pad 8 thru_hole oval (at 0 17.78) (size 1.7 1.7) (drill 1) (layers *.Cu *.Mask)
-      (net 7 /L3))
+      (net 6 /L3))
     (pad 9 thru_hole oval (at 0 20.32) (size 1.7 1.7) (drill 1) (layers *.Cu *.Mask)
-      (net 8 /L4))
+      (net 7 /L4))
     (pad 10 thru_hole oval (at 0 22.86) (size 1.7 1.7) (drill 1) (layers *.Cu *.Mask)
-      (net 9 /L5))
+      (net 8 /L5))
     (pad 11 thru_hole oval (at 0 25.4) (size 1.7 1.7) (drill 1) (layers *.Cu *.Mask)
-      (net 10 /L6))
+      (net 9 /L6))
     (pad 12 thru_hole oval (at 0 27.94) (size 1.7 1.7) (drill 1) (layers *.Cu *.Mask)
-      (net 11 /L7))
+      (net 10 /L7))
     (model ${KISYS3DMOD}/Socket_Strips.3dshapes/Socket_Strip_Straight_1x12_Pitch2.54mm.wrl
       (at (xyz 0 -0.55 0))
@@
     )
     (pad 1 thru_hole rect (at 0 0) (size 1.7 1.7) (drill 1) (layers *.Cu *.Mask)
-      (net 20 /VIN2))
+      (net 19 /VIN2))
     (pad 2 thru_hole oval (at 0 2.54) (size 1.7 1.7) (drill 1) (layers *.Cu *.Mask)
-      (net 21 /VCC2))
+      (net 20 /VCC2))
     (pad 3 thru_hole oval (at 0 5.08) (size 1.7 1.7) (drill 1) (layers *.Cu *.Mask)
-      (net 22 /GND2))
+      (net 21 /GND2))
     (pad 4 thru_hole oval (at 0 7.62) (size 1.7 1.7) (drill 1) (layers *.Cu *.Mask))
     (pad 5 thru_hole oval (at 0 10.16) (size 1.7 1.7) (drill 1) (layers *.Cu *.Mask)
-      (net 12 /D0))
+      (net 11 /D0))
     (pad 6 thru_hole oval (at 0 12.7) (size 1.7 1.7) (drill 1) (layers *.Cu *.Mask)
-      (net 13 /D1))
+      (net 12 /D1))
     (pad 7 thru_hole oval (at 0 15.24) (size 1.7 1.7) (drill 1) (layers *.Cu *.Mask)
-      (net 14 /D2))
+      (net 13 /D2))
     (pad 8 thru_hole oval (at 0 17.78) (size 1.7 1.7) (drill 1) (layers *.Cu *.Mask)
-      (net 15 /D3))
+      (net 14 /D3))
     (pad 9 thru_hole oval (at 0 20.32) (size 1.7 1.7) (drill 1) (layers *.Cu *.Mask)
-      (net 16 /D4))
+      (net 15 /D4))
     (pad 10 thru_hole oval (at 0 22.86) (size 1.7 1.7) (drill 1) (layers *.Cu *.Mask)
-      (net 17 /D5))
+      (net 16 /D5))
     (pad 11 thru_hole oval (at 0 25.4) (size 1.7 1.7) (drill 1) (layers *.Cu *.Mask)
-      (net 18 /D6))
+      (net 17 /D6))
     (pad 12 thru_hole oval (at 0 27.94) (size 1.7 1.7) (drill 1) (layers *.Cu *.Mask)
-      (net 19 /D7))
+      (net 18 /D7))
     (model ${KISYS3DMOD}/Socket_Strips.3dshapes/Socket_Strip_Straight_1x12_Pitch2.54mm.wrl
       (at (xyz 0 -0.55 0))
@@
     )
   )
-  (zone (net 22) (net_name /GND2) (layer B.Cu) (hatch edge 0.508)
+  (zone (net 21) (net_name /GND2) (layer B.Cu) (hatch edge 0.508)
     (connect_pads (clearance 0.508))
     (min_thickness 0.254)
@@
     )
   )
-  (zone (net 3) (net_name Earth) (layer B.Cu) (hatch edge 0.508)
+  (zone (net 22) (net_name /GND) (layer B.Cu) (hatch edge 0.508)
     (connect_pads (clearance 0.508))
     (min_thickness 0.254)
