File: buttons/buttons.kicad_pcb (KiCad board)
At the start: 2 copper layers, 24 parts, among them SW1 SW_Push, SW2 SW_Push, SW3 SW_Push, SW4 SW_Push, SW5 SW_Push, SW6 SW_Push, SW7 SW_Push, SW8 SW_Push

Commit message: More work to ensure there are no errors from KiCAD's schematic checker. Fixed the multiplexer module, so that all 7 slaves will work (only 6 were working, due to a missing VCC to the "Next Output").
Parts:
- H1: value Headers8L -> Choice
- H2: value Headers8 -> Select
Changed lines of the file:
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@@
     (links 67)
     (no_connects 0)
-    (area 124.46 82.55 174.07 132.080001)
+    (area 0 0 0 0)
     (thickness 1.6)
     (drawings 10)
@@
       (effects (font (size 1 1) (thickness 0.15)))
     )
-    (fp_text value Headers8L (at 0 20.11) (layer F.Fab)
+    (fp_text value Choice (at 0 20.11) (layer F.Fab)
       (effects (font (size 1 1) (thickness 0.15)))
     )
@@
       (effects (font (size 1 1) (thickness 0.15)))
     )
-    (fp_text value Headers8 (at 0 20.11) (layer F.Fab)
-      (effects (font (size 1 1) (thickness 0.15)))
-    )
+    (fp_text value Select (at 0 20.11) (layer F.Fab)
+      (effects (font (size 1 1) (thickness 0.15)))
+    )
