File: i2c/i2c.kicad_pcb (KiCad board)
At the start: 2 copper layers, 16 parts, among them J1 Conn_01x05, J2 Conn_01x07, J3 GS2, J4 GS2, J5 GS2

Commit message: More work to ensure there are no errors from KiCAD's schematic checker. Fixed the multiplexer module, so that all 7 slaves will work (only 6 were working, due to a missing VCC to the "Next Output").
Connections:
- net /L1 renamed /MISO
- net /L3 renamed /D10
- net /L6 renamed /TXD
- net /L7 renamed /RXD
- I1 pad 3: Earth -> /GND
- I2C1 pad 1: Earth -> /GND
- I2C2 pad 1: (no net) -> /GND
- I2C3 pad 1: Earth -> /GND
- I2C4 pad 1: Earth -> /GND
- J2 pad 1: Earth -> /GND
- J5 pad 2: Earth -> /GND
- O1 pad 3: Earth -> /GND
Routing:
- net Earth: track 43.8 -> 0.00 mm, vias 1 -> 0
- net /GND: track 0.00 -> 43.8 mm, vias 0 -> 1
- added copper zone on B.Cu, net /GND
- removed copper zone on B.Cu, net Earth
