File: ioExpansion-23017/ioExpansion.sch (KiCad schematic (older format))
At the start: 14 parts, among them J1 GS3, J2 GS3, J3 GS3, J4 Interrupt, U1 MCP23017

Commit message: More work to ensure there are no errors from KiCAD's schematic checker. Fixed the multiplexer module, so that all 7 slaves will work (only 6 were working, due to a missing VCC to the "Next Output").
Parts:
- removed H1: Headers8, Pin_Headers:Pin_Header_Straight_1x08_Pitch2.54mm, symbol Headers8
- removed I2C1, I2C2, I2C3: I2CHeader, Pin_Headers:Pin_Header_Straight_1x04_Pitch2.54mm, symbol I2CHeader-RESCUE-MCP23017
- added I2C1, I2C2, I2C3: I2CHeader, Pin_Headers:Pin_Header_Straight_1x04_Pitch2.54mm, symbol I2CHeader
Connections:
- net GND: now also I2C1.1 (GND), I2C2.1 (GND), I2C3.1 (GND)
- net L4: now also I2C1.4 (SDA), I2C2.4 (SDA), I2C3.4 (SDA)
- net L5: now also I2C1.3 (SCL), I2C2.3 (SCL), I2C3.3 (SCL)
- net VCC: now also I2C1.2 (VCC), I2C2.2 (VCC), I2C3.2 (VCC)
Changed lines of the file:
@@
 LIBS:valves
 LIBS:eplay
-LIBS:Switch
-LIBS:ioExpansion-cache
 EELAYER 25 0
 EELAYER END
@@
 Text Label 4900 3850 0    60   ~ 0
 VCC
-$Comp
-L I2CHeader-RESCUE-MCP23017 I2C1
-U 1 1 5AC33E90
-P 6100 4150
-F 0 "I2C1" H 6250 3750 60  0000 C CNN
-F 1 "I2CHeader" H 6250 4250 60  0000 C CNN
-F 2 "Pin_Headers:Pin_Header_Straight_1x04_Pitch2.54mm" H 5900 4200 60  0001 C CNN
-F 3 "" H 5900 4200 60  0001 C CNN
-	1    6100 4150
-	1    0    0    -1
-$EndComp
 Text Label 5900 4350 2    60   ~ 0
 SCL
@@
 Text Label 5900 4150 2    60   ~ 0
 GND
-$Comp
-L Headers8 H1
-U 1 1 5AC34BA3
-P 5800 2050
-F 0 "H1" H 5800 1000 60  0000 C CNN
-F 1 "Headers8" H 5850 2000 60  0000 C CNN
-F 2 "Pin_Headers:Pin_Header_Straight_1x08_Pitch2.54mm" H 5850 2000 60  0001 C CNN
-F 3 "" H 5850 2000 60  0001 C CNN
-	1    5800 2050
-	1    0    0    -1
-$EndComp
 $Comp
 L GS3 J1
@@
 	1    0    0    -1
 $EndComp
-$Comp
-L I2CHeader-RESCUE-MCP23017 I2C2
-U 1 1 5AE715A1
+Wire Wire Line
+	5900 4150 7200 4150
+Wire Wire Line
+	5900 4250 7200 4250
+Wire Wire Line
+	5900 4350 7200 4350
+Wire Wire Line
+	5900 4450 7200 4450
+Connection ~ 6550 4150
+Connection ~ 6550 4250
+Connection ~ 6550 4350
+Connection ~ 6550 4450
+$Comp
+L I2CHeader I2C3
+U 1 1 5AFEAB9E
+P 7400 4150
+F 0 "I2C3" H 7550 3750 60  0000 C CNN
+F 1 "I2CHeader" H 7550 4250 60  0000 C CNN
+F 2 "Pin_Headers:Pin_Header_Straight_1x04_Pitch2.54mm" H 7200 4200 60  0001 C CNN
+F 3 "" H 7200 4200 60  0001 C CNN
+	1    7400 4150
+	1    0    0    -1
+$EndComp
+$Comp
+L I2CHeader I2C2
+U 1 1 5AFEAC2B
 P 6750 4150
 F 0 "I2C2" H 6900 3750 60  0000 C CNN
@@
 	1    0    0    -1
 $EndComp
-Wire Wire Line
-	5900 4150 7200 4150
-Wire Wire Line
-	5900 4250 7200 4250
-Wire Wire Line
-	5900 4350 7200 4350
-Wire Wire Line
-	5900 4450 7200 4450
-$Comp
-L I2CHeader-RESCUE-MCP23017 I2C3
-U 1 1 5AE717BC
-P 7400 4150
-F 0 "I2C3" H 7550 3750 60  0000 C CNN
-F 1 "I2CHeader" H 7550 4250 60  0000 C CNN
-F 2 "Pin_Headers:Pin_Header_Straight_1x04_Pitch2.54mm" H 7200 4200 60  0001 C CNN
-F 3 "" H 7200 4200 60  0001 C CNN
-	1    7400 4150
-	1    0    0    -1
-$EndComp
-Connection ~ 6550 4150
-Connection ~ 6550 4250
-Connection ~ 6550 4350
-Connection ~ 6550 4450
+$Comp
+L I2CHeader I2C1
+U 1 1 5AFEAC77
+P 6100 4150
+F 0 "I2C1" H 6250 3750 60  0000 C CNN
+F 1 "I2CHeader" H 6250 4250 60  0000 C CNN
+F 2 "Pin_Headers:Pin_Header_Straight_1x04_Pitch2.54mm" H 5900 4200 60  0001 C CNN
+F 3 "" H 5900 4200 60  0001 C CNN
+	1    6100 4150
+	1    0    0    -1
+$EndComp
 $EndSCHEMATC
