File: levelConverter/levelConverter.sch (KiCad schematic (older format))
At the start: 27 parts, among them Q1 BSS138, Q2 BSS138, Q3 BSS138, Q4 BSS138, Q5 BSS138, Q6 BSS138, Q7 BSS138, Q8 BSS138, U1 AP1117-33

Commit message: More work to ensure there are no errors from KiCAD's schematic checker. Fixed the multiplexer module, so that all 7 slaves will work (only 6 were working, due to a missing VCC to the "Next Output").
Connections:
- net Earth renamed GND
Changed lines of the file:
@@
 LIBS:valves
 LIBS:eplay
-LIBS:levelConverter-cache
 EELAYER 25 0
 EELAYER END
@@
 L7
 $Comp
-L Earth #PWR01
-U 1 1 5AC24527
-P 2250 2100
-F 0 "#PWR01" H 2250 1850 50  0001 C CNN
-F 1 "Earth" H 2250 1950 50  0001 C CNN
-F 2 "" H 2250 2100 50  0001 C CNN
-F 3 "" H 2250 2100 50  0001 C CNN
-	1    2250 2100
-	1    0    0    -1
-$EndComp
-$Comp
 L Input I1
 U 1 1 5AC3D559
@@
 Text Label 4100 2000 2    60   ~ 0
 3v3
+$Comp
+L PWR_FLAG #FLG01
+U 1 1 5AFEC326
+P 3650 2000
+F 0 "#FLG01" H 3650 2075 50  0001 C CNN
+F 1 "PWR_FLAG" H 3650 2150 50  0000 C CNN
+F 2 "" H 3650 2000 50  0001 C CNN
+F 3 "" H 3650 2000 50  0001 C CNN
+	1    3650 2000
+	1    0    0    -1
+$EndComp
+Connection ~ 3650 2000
 $EndSCHEMATC
