File: levelConverterAndHeaders/levelConverter.sch (KiCad schematic (older format))
At the start: 22 parts, among them J1 S, J2 Term, J3 S, J4 Term, Q1 BSS138, Q2 BSS138, Q3 BSS138, Q4 BSS138, Q5 BSS138, Q6 BSS138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

Commit message: More work to ensure there are no errors from KiCAD's schematic checker. Fixed the multiplexer module, so that all 7 slaves will work (only 6 were working, due to a missing VCC to the "Next Output").
Parts:
- removed H1: Data, Pin_Headers:Pin_Header_Straight_1x08_Pitch2.54mm, symbol Headers8L
- removed H2: GND, Pin_Headers:Pin_Header_Straight_1x08_Pitch2.54mm, symbol Headers8L
- removed H3: VCC, Pin_Headers:Pin_Header_Straight_1x08_Pitch2.54mm, symbol Headers8L
- added J5: GND, Pin_Headers:Pin_Header_Straight_1x08_Pitch2.54mm, symbol Conn_01x08
- added J6: VCC, Pin_Headers:Pin_Header_Straight_1x08_Pitch2.54mm, symbol Conn_01x08
- added J7: Data, Pin_Headers:Pin_Header_Straight_1x08_Pitch2.54mm, symbol Conn_01x08
Connections:
- net at I2.10 (L5), O2.10 (L5): now also J7.6 (Pin_6)
- net at I2.11 (L6), O2.11 (L6): now also J7.7 (Pin_7)
- net at I2.12 (L7), O2.12 (L7): now also J7.8 (Pin_8)
- net VCC2: now reaches I2.2 (VCC), J2.2 (Pin_2), J4.2 (Pin_2), O2.2 (VCC)
- net VCC2: now also J6.1 (Pin_1), J6.2 (Pin_2), J6.3 (Pin_3), J6.4 (Pin_4), J6.5 (Pin_5), J6.6 (Pin_6), J6.7 (Pin_7), J6.8 (Pin_8)
- net at I2.5 (L0), O2.5 (L0): now also J7.1 (Pin_1)
- net at I2.6 (L1), O2.6 (L1): now also J7.2 (Pin_2)
- net at I2.7 (L2), O2.7 (L2): now also J7.3 (Pin_3)
- net at I2.8 (L3), O2.8 (L3): now also J7.4 (Pin_4)
- net at I2.9 (L4), O2.9 (L4): now also J7.5 (Pin_5)
- net at J3.1 (Pin_1): now also J4.1 (Pin_1); no longer J4.3 (Pin_3)
- removed net Earth: I1.3 (GND), I2.3 (GND), J2.1 (Pin_1), J4.1 (Pin_1), O1.3 (GND), O2.3 (GND), U1.1 (GND)
- new net GND: I1.3 (GND), O1.3 (GND), U1.1 (GND)
- new net GND2: I2.3 (GND), J2.1 (Pin_1), J4.3 (Pin_3), J5.1 (Pin_1), J5.2 (Pin_2), J5.3 (Pin_3), J5.4 (Pin_4), J5.5 (Pin_5), J5.6 (Pin_6), J5.7 (Pin_7), J5.8 (Pin_8), O2.3 (GND)
Other:
- moved on the sheet: J3, J4
Changed lines of the file:
@@
 LIBS:valves
 LIBS:eplay
-LIBS:levelConverter-cache
 EELAYER 25 0
 EELAYER END
@@
 L7
 $Comp
-L Earth #PWR01
-U 1 1 5AC24527
-P 1750 2100
-F 0 "#PWR01" H 1750 1850 50  0001 C CNN
-F 1 "Earth" H 1750 1950 50  0001 C CNN
-F 2 "" H 1750 2100 50  0001 C CNN
-F 3 "" H 1750 2100 50  0001 C CNN
-	1    1750 2100
-	1    0    0    -1
-$EndComp
-$Comp
 L Input I1
 U 1 1 5AC3D559
@@
 	1    0    0    -1
 $EndComp
-$Comp
-L Headers8L H1
-U 1 1 5AE76E66
-P 7550 2050
-F 0 "H1" H 7550 1000 60  0000 C CNN
-F 1 "Data" H 7600 2000 60  0000 C CNN
-F 2 "Pin_Headers:Pin_Header_Straight_1x08_Pitch2.54mm" H 7600 2000 60  0001 C CNN
-F 3 "" H 7600 2000 60  0001 C CNN
-	1    7550 2050
-	1    0    0    -1
-$EndComp
-$Comp
-L Headers8L H2
-U 1 1 5AE76ECE
-P 9300 2050
-F 0 "H2" H 9300 1000 60  0000 C CNN
-F 1 "GND" H 9350 2000 60  0000 C CNN
-F 2 "Pin_Headers:Pin_Header_Straight_1x08_Pitch2.54mm" H 9350 2000 60  0001 C CNN
-F 3 "" H 9350 2000 60  0001 C CNN
-	1    9300 2050
-	1    0    0    -1
-$EndComp
-$Comp
-L Headers8L H3
-U 1 1 5AE76F97
-P 9750 2050
-F 0 "H3" H 9750 1000 60  0000 C CNN
-F 1 "VCC" H 9800 2000 60  0000 C CNN
-F 2 "Pin_Headers:Pin_Header_Straight_1x08_Pitch2.54mm" H 9800 2000 60  0001 C CNN
-F 3 "" H 9800 2000 60  0001 C CNN
-	1    9750 2050
-	1    0    0    -1
-$EndComp
 Wire Wire Line
 	3300 2300 4800 2300
@@
 	7250 1900 8300 1900
 Wire Wire Line
-	7250 2000 9650 2000
+	7250 2000 9450 2000
 Wire Wire Line
 	7250 2100 9000 2100
 Wire Wire Line
-	8300 2300 7250 2300
+	7250 2300 8300 2300
 Wire Wire Line
 	7250 2400 8300 2400
 Wire Wire Line
-	8300 2500 7250 2500
+	7250 2500 8300 2500
 Wire Wire Line
 	7250 2600 8300 2600
 Wire Wire Line
-	8300 2700 7250 2700
+	7250 2700 8300 2700
 Wire Wire Line
 	7250 2800 8300 2800
 Wire Wire Line
-	8300 2900 7250 2900
+	7250 2900 8300 2900
 Wire Wire Line
 	7250 3000 8300 3000
@@
 Connection ~ 9450 2400
 Wire Wire Line
-	9450 2000 9450 3250
+	9450 1650 9450 3250
 Text Label 7950 2100 0    60   ~ 0
-GND
+GND2
 Connection ~ 9000 2300
 Connection ~ 8300 2000
@@
 	2700 2800 2900 2800
 Wire Wire Line
-	2900 3300 2600 3300
-Wire Wire Line
-	2600 3300 2600 1900
+	2600 3300 2900 3300
+Wire Wire Line
+	2600 1900 2600 3300
 Wire Wire Line
 	2500 1900 2500 3800
@@
 	2500 3800 2900 3800
 Wire Wire Line
-	2400 4300 2400 1900
-Wire Wire Line
-	2900 4300 2400 4300
-Wire Wire Line
-	2900 4800 2300 4800
-Wire Wire Line
-	2300 4800 2300 1900
-Wire Wire Line
-	2900 5350 2200 5350
-Wire Wire Line
-	2200 5350 2200 1900
+	2400 1900 2400 4300
+Wire Wire Line
+	2400 4300 2900 4300
+Wire Wire Line
+	2300 4800 2900 4800
+Wire Wire Line
+	2300 1900 2300 4800
+Wire Wire Line
+	2200 5350 2900 5350
+Wire Wire Line
+	2200 1900 2200 5350
 Wire Wire Line
 	2100 1900 2100 5950
@@
 	9200 3450 9550 3450
 Text Label 9750 3450 0    60   ~ 0
-GND
+GND2
 $Comp
 L Conn_01x01 J3
 U 1 1 5AE82489
-P 9300 1850
-F 0 "J3" H 9300 1950 50  0000 C CNN
-F 1 "S" H 9300 1750 50  0000 C CNN
-F 2 "Pin_Headers:Pin_Header_Straight_1x01_Pitch2.54mm" H 9300 1850 50  0001 C CNN
-F 3 "" H 9300 1850 50  0001 C CNN
-	1    9300 1850
+P 9350 1850
+F 0 "J3" H 9350 1950 50  0000 C CNN
+F 1 "S" H 9350 1750 50  0000 C CNN
+F 2 "Pin_Headers:Pin_Header_Straight_1x01_Pitch2.54mm" H 9350 1850 50  0001 C CNN
+F 3 "" H 9350 1850 50  0001 C CNN
+	1    9350 1850
 	0    1    1    0
 $EndComp
@@
 L Conn_01x03 J4
 U 1 1 5AE82510
-P 9650 1850
-F 0 "J4" H 9650 2050 50  0000 C CNN
-F 1 "Term" H 9650 1650 50  0000 C CNN
-F 2 "Connectors_Terminal_Blocks:TerminalBlock_Pheonix_MPT-2.54mm_3pol" H 9650 1850 50  0001 C CNN
-F 3 "" H 9650 1850 50  0001 C CNN
-	1    9650 1850
-	0    1    1    0
-$EndComp
-Text Label 9750 1650 0    60   ~ 0
-GND
-Wire Wire Line
-	9550 1650 9300 1650
-Wire Wire Line
-	9650 2000 9650 1650
+P 9450 1450
+F 0 "J4" H 9450 1650 50  0000 C CNN
+F 1 "Term" H 9450 1250 50  0000 C CNN
+F 2 "Connectors_Terminal_Blocks:TerminalBlock_Pheonix_MPT-2.54mm_3pol" H 9450 1450 50  0001 C CNN
+F 3 "" H 9450 1450 50  0001 C CNN
+	1    9450 1450
+	0    -1   -1   0
+$EndComp
+Text Label 9550 1650 0    60   ~ 0
+GND2
 Connection ~ 9450 2000
 Wire Wire Line
@@
 Text Notes 9950 3950 2    60   ~ 0
 Option for one triple\nusing screw terminal
-Text Notes 9950 1550 2    60   ~ 0
+Text Notes 9950 1300 2    60   ~ 0
 Option for one triple\nusing screw terminal
+$Comp
+L Conn_01x08 J5
+U 1 1 5AFEC944
+P 9200 2600
+F 0 "J5" H 9200 3000 50  0000 C CNN
+F 1 "GND" H 9200 2100 50  0000 C CNN
+F 2 "Pin_Headers:Pin_Header_Straight_1x08_Pitch2.54mm" H 9200 2600 50  0001 C CNN
+F 3 "" H 9200 2600 50  0001 C CNN
+	1    9200 2600
+	1    0    0    -1
+$EndComp
+$Comp
+L Conn_01x08 J6
+U 1 1 5AFEC9E1
+P 9650 2600
+F 0 "J6" H 9650 3000 50  0000 C CNN
+F 1 "VCC" H 9650 2100 50  0000 C CNN
+F 2 "Pin_Headers:Pin_Header_Straight_1x08_Pitch2.54mm" H 9650 2600 50  0001 C CNN
+F 3 "" H 9650 2600 50  0001 C CNN
+	1    9650 2600
+	1    0    0    -1
+$EndComp
+$Comp
+L PWR_FLAG #FLG01
+U 1 1 5AFECBDF
+P 4400 1350
+F 0 "#FLG01" H 4400 1425 50  0001 C CNN
+F 1 "PWR_FLAG" H 4400 1500 50  0000 C CNN
+F 2 "" H 4400 1350 50  0001 C CNN
+F 3 "" H 4400 1350 50  0001 C CNN
+	1    4400 1350
+	1    0    0    -1
+$EndComp
+Text Label 7950 2000 0    60   ~ 0
+VCC2
+$Comp
+L Conn_01x08 J7
+U 1 1 5AFED967
+P 7850 2600
+F 0 "J7" H 7850 3000 50  0000 C CNN
+F 1 "Data" H 7850 2100 50  0000 C CNN
+F 2 "Pin_Headers:Pin_Header_Straight_1x08_Pitch2.54mm" H 7850 2600 50  0001 C CNN
+F 3 "" H 7850 2600 50  0001 C CNN
+	1    7850 2600
+	1    0    0    -1
+$EndComp
+Connection ~ 7650 2300
+Connection ~ 7650 2400
+Connection ~ 7650 2500
+Connection ~ 7650 2600
+Connection ~ 7650 2700
+Connection ~ 7650 2800
+Connection ~ 7650 2900
+Connection ~ 7650 3000
 $EndSCHEMATC
