File: multiplexer/multiplxer.sch (KiCad schematic (older format))
At the start: 10 parts, among them J1 Conn_01x04, U1 74HC595, U2 4051

Commit message: More work to ensure there are no errors from KiCAD's schematic checker. Fixed the multiplexer module, so that all 7 slaves will work (only 6 were working, due to a missing VCC to the "Next Output").
Parts:
- removed H1: Headers8L, Pin_Headers:Pin_Header_Straight_1x08_Pitch2.54mm, symbol Headers8L
- added J2: Choice, Pin_Headers:Pin_Header_Straight_1x08_Pitch2.54mm, symbol Conn_01x08
- I1: value Input -> Master Input
- I2: value Input -> Prev Input
- J1: value Conn_01x04 -> Select
- O2: value Output -> Next Output
Connections:
- net L0: now also J2.1 (Pin_1)
- net L1: now also J2.2 (Pin_2)
- net L2: now also J2.3 (Pin_3)
- net L3: now also J2.4 (Pin_4)
- net L4: now also J2.5 (Pin_5)
- net L5: now also J2.6 (Pin_6)
- net L6: now also J2.7 (Pin_7)
- net L7: now also J2.8 (Pin_8)
- net VCC: now also O2.12 (L7)
- no-connect marks 2 -> 1
Other:
- note added: "ERRORS.\nThe two configurations, means there are 3 errors\nreported by KiCAD, which I don't know how to avoid.\nOnly I1 or I2 will be populated, so there is no problems\nin the actual boards."
Changed lines of the file:
@@
 LIBS:valves
 LIBS:eplay
-LIBS:multiplxer-cache
 EELAYER 25 0
 EELAYER END
@@
 P 1950 1600
 F 0 "I1" H 1950 50  60  0000 C CNN
-F 1 "Input" H 2000 1550 60  0000 C CNN
+F 1 "Master Input" H 2000 1550 60  0000 C CNN
 F 2 "Pin_Headers:Pin_Header_Straight_1x12_Pitch2.54mm" H 2000 1550 60  0001 C CNN
 F 3 "" H 2000 1550 60  0001 C CNN
@@
 Text Label 7150 4050 2    60   ~ 0
 GND
-$Comp
-L Headers8L H1
-U 1 1 5ACC6450
-P 3100 2050
-F 0 "H1" H 3100 1000 60  0000 C CNN
-F 1 "Headers8L" H 3150 2000 60  0000 C CNN
-F 2 "Pin_Headers:Pin_Header_Straight_1x08_Pitch2.54mm" H 3150 2000 60  0001 C CNN
-F 3 "" H 3150 2000 60  0001 C CNN
-	1    3100 2050
-	1    0    0    -1
-$EndComp
 Text Label 4400 2850 2    60   ~ 0
 VCC
@@
 P 7450 1850
 F 0 "O2" H 7450 300 60  0000 C CNN
-F 1 "Output" H 7350 1800 60  0000 C CNN
+F 1 "Next Output" H 7350 1800 60  0000 C CNN
 F 2 "Socket_Strips:Socket_Strip_Straight_1x12_Pitch2.54mm" H 7500 1800 60  0001 C CNN
 F 3 "" H 7500 1800 60  0001 C CNN
@@
 P 5400 650
 F 0 "I2" H 5400 -900 60  0000 C CNN
-F 1 "Input" H 5450 600 60  0000 C CNN
+F 1 "Prev Input" H 5450 600 60  0000 C CNN
 F 2 "Pin_Headers:Pin_Header_Straight_1x12_Pitch2.54mm" H 5450 600 60  0001 C CNN
 F 3 "" H 5450 600 60  0001 C CNN
@@
 P 3700 2750
 F 0 "J1" H 3700 2950 50  0000 C CNN
-F 1 "Conn_01x04" H 3700 2450 50  0000 C CNN
+F 1 "Select" H 3700 2450 50  0000 C CNN
 F 2 "Pin_Headers:Pin_Header_Straight_1x04_Pitch2.54mm" H 3700 2750 50  0001 C CNN
 F 3 "" H 3700 2750 50  0001 C CNN
@@
 VSS
 NoConn ~ 5800 3450
-NoConn ~ 7150 3250
+$Comp
+L Conn_01x08 J2
+U 1 1 5AFECC5F
+P 3000 2600
+F 0 "J2" H 3000 3000 50  0000 C CNN
+F 1 "Choice" H 3000 2100 50  0000 C CNN
+F 2 "Pin_Headers:Pin_Header_Straight_1x08_Pitch2.54mm" H 3000 2600 50  0001 C CNN
+F 3 "" H 3000 2600 50  0001 C CNN
+	1    3000 2600
+	1    0    0    -1
+$EndComp
+Text Notes 1950 1100 0    60   ~ 0
+ERRORS.\nThe two configurations, means there are 3 errors\nreported by KiCAD, which I don't know how to avoid.\nOnly I1 or I2 will be populated, so there is no problems\nin the actual boards.
+Text Label 7150 3250 2    60   ~ 0
+VCC
 $EndSCHEMATC
