File: proMini/proMini.kicad_pcb (KiCad board)
At the start: 2 copper layers, 10 parts

Commit message: More update to make the libraryies use only relative paths.
Parts:
- removed FT1, FT2: FTDI, Pin_Headers:Pin_Header_Straight_1x06_Pitch2.54mm
- added J1: ICSP, Pin_Headers:Pin_Header_Straight_1x06_Pitch2.54mm, F.Cu at (111.8, 58.4)
- added J2: ICSP, Pin_Headers:Pin_Header_Straight_1x06_Pitch2.54mm, F.Cu at (111.8, 40.6)
Changed lines of the file:
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@@
     (links 48)
     (no_connects 0)
-    (area 108.585 31.115 158.115001 80.645001)
+    (area 0 0 0 0)
     (thickness 1.6)
     (drawings 41)
@@
     (descr "Through hole straight pin header, 1x06, 2.54mm pitch, single row")
     (tags "Through hole pin header THT 1x06 2.54mm single row")
-    (fp_text reference FT1 (at 0 -2.33) (layer F.Fab)
-      (effects (font (size 1 1) (thickness 0.15)))
-    )
-    (fp_text value FTDI (at 0 15.03) (layer F.Fab)
+    (fp_text reference J1 (at 0 -2.33) (layer F.SilkS)
+      (effects (font (size 1 1) (thickness 0.15)))
+    )
+    (fp_text value ICSP (at 0 15.03) (layer F.Fab)
       (effects (font (size 1 1) (thickness 0.15)))
     )
@@
     (descr "Through hole straight pin header, 1x06, 2.54mm pitch, single row")
     (tags "Through hole pin header THT 1x06 2.54mm single row")
-    (fp_text reference FT2 (at 0 -2.33) (layer F.Fab)
-      (effects (font (size 1 1) (thickness 0.15)))
-    )
-    (fp_text value FTDI (at 0 15.03) (layer F.Fab)
-      (effects (font (size 1 1) (thickness 0.15)))
-    )
+    (fp_text reference J2 (at 0 -2.33) (layer F.SilkS)
+      (effects (font (size 1 1) (thickness 0.15)))
+    )
+    (fp_text value ICSP (at 0 15.03) (layer F.Fab)
+      (effects (font (size 1 1) (thickness 0.15)))
+    )
