File: prototype/prototype.kicad_pcb (KiCad board)
At the start: 2 copper layers, 39 parts, among them J1 GS2, J10 Conn_01x14, J11 Conn_01x14, J12 Conn_01x08, J13 Conn_01x08, J2 GS2, J3 GS2, J4 GS2, J5 GS2, J6 GS2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

Commit message: More update to make the libraryies use only relative paths.
Parts:
- removed H1: Headers8L, Pin_Headers:Pin_Header_Straight_1x08_Pitch2.54mm
- removed H4: Headers8, Pin_Headers:Pin_Header_Straight_1x08_Pitch2.54mm
- added J14: IN Data, Pin_Headers:Pin_Header_Straight_1x08_Pitch2.54mm, F.Cu at (128.9, 102.9)
- added J15: Out Data, Pin_Headers:Pin_Header_Straight_1x08_Pitch2.54mm, F.Cu at (164.5, 120.7)
- J10: value Conn_01x14 -> VCC
- J11: value Conn_01x14 -> VIN
- J12: value Conn_01x08 -> Out Data; moved to F.Cu
- J13: value Conn_01x08 -> IN Data; moved to F.Cu
- J9: value Conn_01x14 -> GND
- turned J12 to 90 degrees
- turned J13 to 90 degrees
Connections:
- net Earth renamed /GND
