File: prototype/prototype.sch (KiCad schematic (older format))
At the start: 19 parts, among them J1 GS2, J10 Conn_01x14, J11 Conn_01x14, J12 Conn_01x08, J13 Conn_01x08, J2 GS2, J3 GS2, J4 GS2, J5 GS2, J6 GS2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

Commit message: More update to make the libraryies use only relative paths.
Parts:
- removed H1: Headers8L, Pin_Headers:Pin_Header_Straight_1x08_Pitch2.54mm, symbol Headers8L
- removed H4: Headers8, Pin_Headers:Pin_Header_Straight_1x08_Pitch2.54mm, symbol Headers8
- added J14: IN Data, Pin_Headers:Pin_Header_Straight_1x08_Pitch2.54mm, symbol Conn_01x08
- added J15: Out Data, Pin_Headers:Pin_Header_Straight_1x08_Pitch2.54mm, symbol Conn_01x08
- J10: value Conn_01x14 -> VCC
- J11: value Conn_01x14 -> VIN
- J12: value Conn_01x08 -> Out Data
- J13: value Conn_01x08 -> IN Data
- J9: value Conn_01x14 -> GND
Connections:
- net L0: now also J14.1 (Pin_1)
- net L1: now also J14.2 (Pin_2)
- net L2: now also J14.3 (Pin_3)
- net L3: now also J14.4 (Pin_4)
- net L4: now also J14.5 (Pin_5)
- net L5: now also J14.6 (Pin_6)
- net L6: now also J14.7 (Pin_7)
- net L7: now also J14.8 (Pin_8)
- net at J6.1 (G1), O2.10 (L5): now also J15.3 (Pin_3)
- net at J7.1 (G1), O2.11 (L6): now also J15.2 (Pin_2)
- net at J8.1 (G1), O2.12 (L7): now also J15.1 (Pin_1)
- net at J1.1 (G1), O2.5 (L0): now also J15.8 (Pin_8)
- net at J2.1 (G1), O2.6 (L1): now also J15.7 (Pin_7)
- net at J3.1 (G1), O2.7 (L2): now also J15.6 (Pin_6)
- net at J4.1 (G1), O2.8 (L3): now also J15.5 (Pin_5)
- net at J5.1 (G1), O2.9 (L4): now also J15.4 (Pin_4)
- net Earth renamed GND
Other:
- moved on the sheet: I2, J12, J13, O1
Changed lines of the file:
@@
 L7
-$Comp
-L Earth #PWR01
-U 1 1 5AC24527
-P 2250 2100
-F 0 "#PWR01" H 2250 1850 50  0001 C CNN
-F 1 "Earth" H 2250 1950 50  0001 C CNN
-F 2 "" H 2250 2100 50  0001 C CNN
-F 3 "" H 2250 2100 50  0001 C CNN
-	1    2250 2100
-	1    0    0    -1
-$EndComp
 $Comp
 L Input I1
@@
 L Output O1
 U 1 1 5AC3D61D
-P 4800 5950
-F 0 "O1" H 4800 4400 60  0000 C CNN
-F 1 "Output" H 4700 5900 60  0000 C CNN
-F 2 "Socket_Strips:Socket_Strip_Straight_1x12_Pitch2.54mm" H 4850 5900 60  0001 C CNN
-F 3 "" H 4850 5900 60  0001 C CNN
-	1    4800 5950
-	0    1    1    0
+P 5100 4550
+F 0 "O1" H 5100 3000 60  0000 C CNN
+F 1 "Output" H 5000 4500 60  0000 C CNN
+F 2 "Socket_Strips:Socket_Strip_Straight_1x12_Pitch2.54mm" H 5150 4500 60  0001 C CNN
+F 3 "" H 5150 4500 60  0001 C CNN
+	1    5100 4550
+	1    0    0    -1
 $EndComp
 Text Label 3900 1900 2    60   ~ 0
@@
 Text Label 3900 2100 2    60   ~ 0
 GND
-Text Label 4500 4250 3    60   ~ 0
+Text Label 3400 4850 0    60   ~ 0
 VIN
-Text Label 4400 4250 3    60   ~ 0
+Text Label 3400 4950 0    60   ~ 0
 VCC
-Text Label 4300 4250 3    60   ~ 0
+Text Label 3400 5050 0    60   ~ 0
 GND
 $Comp
 L Input I2
 U 1 1 5AC76C5E
-P 4800 3950
-F 0 "I2" H 4800 2400 60  0000 C CNN
-F 1 "Input" H 4850 3900 60  0000 C CNN
-F 2 "Pin_Headers:Pin_Header_Straight_1x12_Pitch2.54mm" H 4850 3900 60  0001 C CNN
-F 3 "" H 4850 3900 60  0001 C CNN
-	1    4800 3950
-	0    1    1    0
-$EndComp
-$Comp
-L Headers8L H1
-U 1 1 5AC78C62
-P 2550 2050
-F 0 "H1" H 2550 1000 60  0000 C CNN
-F 1 "Headers8L" H 2600 2000 60  0000 C CNN
-F 2 "Pin_Headers:Pin_Header_Straight_1x08_Pitch2.54mm" H 2600 2000 60  0001 C CNN
-F 3 "" H 2600 2000 60  0001 C CNN
-	1    2550 2050
-	1    0    0    -1
-$EndComp
-$Comp
-L Headers8 H4
-U 1 1 5AC79014
-P 3600 2050
-F 0 "H4" H 3600 1000 60  0000 C CNN
-F 1 "Headers8" H 3650 2000 60  0000 C CNN
-F 2 "Pin_Headers:Pin_Header_Straight_1x08_Pitch2.54mm" H 3650 2000 60  0001 C CNN
-F 3 "" H 3650 2000 60  0001 C CNN
-	1    3600 2050
+P 3100 4550
+F 0 "I2" H 3100 3000 60  0000 C CNN
+F 1 "Input" H 3150 4500 60  0000 C CNN
+F 2 "Pin_Headers:Pin_Header_Straight_1x12_Pitch2.54mm" H 3150 4500 60  0001 C CNN
+F 3 "" H 3150 4500 60  0001 C CNN
+	1    3100 4550
 	1    0    0    -1
 $EndComp
@@
 P 5350 2350
 F 0 "J9" H 5350 3050 50  0000 C CNN
-F 1 "Conn_01x14" H 5350 1550 50  0000 C CNN
+F 1 "GND" H 5350 1550 50  0000 C CNN
 F 2 "Pin_Headers:Pin_Header_Straight_1x14_Pitch2.54mm" H 5350 2350 50  0001 C CNN
 F 3 "" H 5350 2350 50  0001 C CNN
@@
 P 5900 2350
 F 0 "J10" H 5900 3050 50  0000 C CNN
-F 1 "Conn_01x14" H 5900 1550 50  0000 C CNN
+F 1 "VCC" H 5900 1550 50  0000 C CNN
 F 2 "Pin_Headers:Pin_Header_Straight_1x14_Pitch2.54mm" H 5900 2350 50  0001 C CNN
 F 3 "" H 5900 2350 50  0001 C CNN
@@
 P 6600 2350
 F 0 "J11" H 6600 3050 50  0000 C CNN
-F 1 "Conn_01x14" H 6600 1550 50  0000 C CNN
+F 1 "VIN" H 6600 1550 50  0000 C CNN
 F 2 "Pin_Headers:Pin_Header_Straight_1x14_Pitch2.54mm" H 6600 2350 50  0001 C CNN
 F 3 "" H 6600 2350 50  0001 C CNN
@@
 VIN
 Wire Wire Line
-	4100 4250 4100 4500
-Wire Wire Line
-	4000 4250 4000 4500
-Wire Wire Line
-	3900 4500 3900 4250
-Wire Wire Line
-	3800 4250 3800 4500
-Wire Wire Line
-	3700 4250 3700 4500
-Wire Wire Line
-	3600 4500 3600 4250
-Wire Wire Line
-	3500 4250 3500 4500
-Wire Wire Line
-	3400 4500 3400 4250
-Text Label 4300 5650 1    60   ~ 0
+	3400 5250 3650 5250
+Wire Wire Line
+	3400 5350 3650 5350
+Wire Wire Line
+	3650 5450 3400 5450
+Wire Wire Line
+	3400 5550 3650 5550
+Wire Wire Line
+	3400 5650 3650 5650
+Wire Wire Line
+	3650 5750 3400 5750
+Wire Wire Line
+	3400 5850 3650 5850
+Wire Wire Line
+	3650 5950 3400 5950
+Text Label 4800 5050 2    60   ~ 0
 GND
-Text Label 4400 5650 1    60   ~ 0
+Text Label 4800 4950 2    60   ~ 0
 VCC
-Text Label 4500 5650 1    60   ~ 0
+Text Label 4800 4850 2    60   ~ 0
 VIN
 Wire Wire Line
-	3400 5650 3400 5200
-Wire Wire Line
-	3500 5200 3500 5650
-Wire Wire Line
-	3600 5650 3600 5200
-Wire Wire Line
-	3700 5200 3700 5650
-Wire Wire Line
-	3800 5650 3800 5200
-Wire Wire Line
-	3900 5200 3900 5650
-Wire Wire Line
-	4000 5650 4000 5200
-Wire Wire Line
-	4100 5200 4100 5650
+	4800 5950 4350 5950
+Wire Wire Line
+	4350 5850 4800 5850
+Wire Wire Line
+	4800 5750 4350 5750
+Wire Wire Line
+	4350 5650 4800 5650
+Wire Wire Line
+	4800 5550 4350 5550
+Wire Wire Line
+	4350 5450 4800 5450
+Wire Wire Line
+	4800 5350 4350 5350
+Wire Wire Line
+	4350 5250 4800 5250
 $Comp
 L Conn_01x08 J13
 U 1 1 5ACF23E1
-P 3800 4700
-F 0 "J13" H 3800 5100 50  0000 C CNN
-F 1 "Conn_01x08" H 3800 4200 50  0000 C CNN
-F 2 "Pin_Headers:Pin_Header_Straight_1x08_Pitch2.54mm" H 3800 4700 50  0001 C CNN
-F 3 "" H 3800 4700 50  0001 C CNN
-	1    3800 4700
-	0    1    1    0
+P 3850 5550
+F 0 "J13" H 3850 5950 50  0000 C CNN
+F 1 "IN Data" H 3850 5050 50  0000 C CNN
+F 2 "Pin_Headers:Pin_Header_Straight_1x08_Pitch2.54mm" H 3850 5550 50  0001 C CNN
+F 3 "" H 3850 5550 50  0001 C CNN
+	1    3850 5550
+	1    0    0    -1
 $EndComp
 $Comp
 L Conn_01x08 J12
 U 1 1 5ACF24E2
-P 3700 5000
-F 0 "J12" H 3700 5400 50  0000 C CNN
-F 1 "Conn_01x08" H 3700 4500 50  0000 C CNN
-F 2 "Pin_Headers:Pin_Header_Straight_1x08_Pitch2.54mm" H 3700 5000 50  0001 C CNN
-F 3 "" H 3700 5000 50  0001 C CNN
-	1    3700 5000
-	0    -1   -1   0
+P 4150 5650
+F 0 "J12" H 4150 6050 50  0000 C CNN
+F 1 "Out Data" H 4150 5150 50  0000 C CNN
+F 2 "Pin_Headers:Pin_Header_Straight_1x08_Pitch2.54mm" H 4150 5650 50  0001 C CNN
+F 3 "" H 4150 5650 50  0001 C CNN
+	1    4150 5650
+	-1   0    0    1
+$EndComp
+$Comp
+L Conn_01x08 J14
+U 1 1 5AFEFE93
+P 2450 2600
+F 0 "J14" H 2450 3000 50  0000 C CNN
+F 1 "IN Data" H 2450 2100 50  0000 C CNN
+F 2 "Pin_Headers:Pin_Header_Straight_1x08_Pitch2.54mm" H 2450 2600 50  0001 C CNN
+F 3 "" H 2450 2600 50  0001 C CNN
+	1    2450 2600
+	1    0    0    -1
+$EndComp
+$Comp
+L Conn_01x08 J15
+U 1 1 5AFEFF4A
+P 3700 2700
+F 0 "J15" H 3700 3100 50  0000 C CNN
+F 1 "Out Data" H 3700 2200 50  0000 C CNN
+F 2 "Pin_Headers:Pin_Header_Straight_1x08_Pitch2.54mm" H 3700 2700 50  0001 C CNN
+F 3 "" H 3700 2700 50  0001 C CNN
+	1    3700 2700
+	-1   0    0    1
 $EndComp
 $EndSCHEMATC
