File: rotaryEncoder/rotaryEncoder.kicad_pcb (KiCad board)
At the start: 2 copper layers, 16 parts, among them J1 Select

Commit message: More update to make the libraryies use only relative paths.
Connections:
- net Earth renamed /GND
